File: omykb-old/omykb.kicad_sch (KiCad schematic)
At the start: 183 parts, among them J2 USB_C_Receptacle_USB2.0_16P, K0 Esc, K1 !,1, K10 ),0, K11 _,-, K12 +,=, K13 Backspace, K14 Home, K15 Tab, K16 Q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

Commit message: trying again
Parts:
- D0, D1, D10, D11, D12, D13, D14, D15, D16, D17, D18, D19, D2, D20, D21, D22, D23, D24, D25, D26, D27, D28, D29, D3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: value D -> 1N4148WS; footprint Diode_SMD:D_0805_2012Metric_Pad1.15x1.40mm_HandSolder -> Diode_SMD:D_SOD-323_HandSoldering
- K33: value D -> Key_D
