File: mykb/mykb.kicad_pcb (KiCad board)
At the start: 2 copper layers, 155 parts, among them J1 USB_mini_micro_B, J2 Conn_02x03_Odd_Even, K0 Esc, K1 !,1, K10 ),0, K11 _,-, K12 +,=, K13 Backspace, K14 Home, K15 Tab, K16 Q, K17 W, K18 E, K19 R, K2 @,2, K20 T, K21 Y, K22 U, K23 I, K24 O, K25 P, K26 {,[, K27 },], K28 |,\, K29 PgUp, K3 #,3, K30 Caps Lock, K31 A, K32 S, K33 D, K34 F, K35 G, K36 H, K37 J, K38 K, K39 L, K4 $,4, K40 :,;, K41 ",', K42 Enter, K43 PgDn, K44 Shift, K45 Z, K46 X, K47 C, K48 V, K49 B, K5 %,5, K50 N, K51 M, K52 <,,, K53 >,., K54 ?,/, K55 Shift, K56 ↑, K57 End, K58 Ctrl, K59 Cmd, K6 ^,6, K60 Alt, K61 Blank, K62 Alt, K63 Ctrl, K64 ←, K65 ↓, K66 →, K7 &,7, K8 *,8, K9 (,9, SW1 SW_Push, U1 ATmega32U4-AU, Y1 Crystal

Commit message: progress on the redo
Parts:
- removed J2: Conn_02x03_Odd_Even, Connector_PinHeader_2.54mm:PinHeader_2x03_P2.54mm_Vertical
- added ?: , , F.Cu at (350.5, 92.5)
- added ?: , , F.Cu at (349.2, 92.5)
- added ?: , , F.Cu at (351.8, 92.5)
- added ?: , , F.Cu at (351.8, 91.3)
- added ?: , , F.Cu at (351.8, 93.8)
- added ?: , , F.Cu at (349.2, 91.3)
- added ?: , , F.Cu at (349.2, 93.8)
- added ?: , , F.Cu at (350.5, 91.3)
- added ?: , , F.Cu at (350.5, 93.8)
- added C10: 100n, Capacitor_SMD:C_0402_1005Metric, F.Cu at (351.6, 99.5)
- added C11: 100n, Capacitor_SMD:C_0402_1005Metric, F.Cu at (343.7, 89.2)
- added C12: 100n, Capacitor_SMD:C_0402_1005Metric, F.Cu at (344.8, 89.2)
- added C13: 100n, Capacitor_SMD:C_0402_1005Metric, F.Cu at (345.9, 89.2)
- added C14: 10uF, Capacitor_SMD:C_0805_2012Metric, F.Cu at (296.9, 94.2)
- added C15: 0.1uf, Capacitor_SMD:C_0603_1608Metric, F.Cu at (329.2, 89.2)
- added C16: 10uF, Capacitor_SMD:C_0805_2012Metric, F.Cu at (286.7, 93.5)
- added C9: 100n, Capacitor_SMD:C_0402_1005Metric, F.Cu at (357.8, 90.3)
- added R10: 10k, Resistor_SMD:R_0603_1608Metric, F.Cu at (332.5, 96.4)
- added R11: 10k, Resistor_SMD:R_0603_1608Metric, F.Cu at (335.5, 96.4)
- added R12: 10k, Resistor_SMD:R_0603_1608Metric, F.Cu at (338.5, 96.4)
- added R13: 10k, Resistor_SMD:R_0603_1608Metric, F.Cu at (341.5, 96.4)
- added R14: 10k, Resistor_SMD:R_0603_1608Metric, F.Cu at (344.5, 96.4)
- added R15: 10k, Resistor_SMD:R_0603_1608Metric, F.Cu at (332.3, 102.5)
- added R16: 10k, Resistor_SMD:R_0603_1608Metric, F.Cu at (335.2, 102.5)
- added R17: 10k, Resistor_SMD:R_0603_1608Metric, F.Cu at (338.2, 102.5)
- added R18: 10k, Resistor_SMD:R_0603_1608Metric, F.Cu at (341.2, 102.5)
- added R19: 10k, Resistor_SMD:R_0603_1608Metric, F.Cu at (354.8, 98.5)
- added R20: 10k, Resistor_SMD:R_0603_1608Metric, F.Cu at (357.8, 98.5)
- added R21: 10k, Resistor_SMD:R_0603_1608Metric, F.Cu at (357.7, 101.4)
- added R22: 10k, Resistor_SMD:R_0603_1608Metric, F.Cu at (360.7, 101.4)
- added R5: 5.1k, Resistor_SMD:R_0603_1608Metric, F.Cu at (305.0, 93.6)
- added R6: 5.1k, Resistor_SMD:R_0603_1608Metric, F.Cu at (305.0, 95.3)
- added R7: 1k, Resistor_SMD:R_0603_1608Metric, F.Cu at (327.7, 89.2)
- added R8: 10k, Resistor_SMD:R_0603_1608Metric, F.Cu at (326.5, 96.4)
- added R9: 10k, Resistor_SMD:R_0603_1608Metric, F.Cu at (329.5, 96.4)
- added SW2: SW_Push, Button_Switch_SMD:SW_Push_1P1T_NO_CK_KMR2, F.Cu at (322.7, 92.8)
- added SW3: RotaryEncoder_Switch_MP, Rotary_Encoder:RotaryEncoder_Alps_EC11E-Switch_Vertical_H20mm, F.Cu at (108.5, 86.8)
- added SW4: RotaryEncoder_Switch_MP, Rotary_Encoder:RotaryEncoder_Alps_EC11E-Switch_Vertical_H20mm, F.Cu at (86.5, 86.8)
- added U2: W25Q128JVS, Package_SO:SOIC-8_5.23x5.23mm_P1.27mm, F.Cu at (334.8, 87.1)
- added U3: NCP1117-3.3_SOT223, Package_TO_SOT_SMD:SOT-223-3_TabPin2, F.Cu at (291.7, 91.3)
- C1, C2: value 0.1u -> 16pF; footprint Capacitor_SMD:C_0805_2012Metric_Pad1.15x1.40mm_HandSolder -> Capacitor_SMD:C_0402_1005Metric; moved to F.Cu
- C3, C4: value 0.1u -> 100n; footprint Capacitor_SMD:C_0805_2012Metric_Pad1.15x1.40mm_HandSolder -> Capacitor_SMD:C_0402_1005Metric; moved to F.Cu
- C5: value 4.7u -> 1u; footprint Capacitor_SMD:C_0805_2012Metric_Pad1.15x1.40mm_HandSolder -> Capacitor_SMD:C_0402_1005Metric; moved to F.Cu
- C6: value 22p -> 1u; footprint Capacitor_SMD:C_0805_2012Metric_Pad1.15x1.40mm_HandSolder -> Capacitor_SMD:C_0402_1005Metric; moved to F.Cu
- C7: value 22p -> 100n; footprint Capacitor_SMD:C_0805_2012Metric_Pad1.15x1.40mm_HandSolder -> Capacitor_SMD:C_0402_1005Metric; moved to F.Cu
- C8: value 1u -> 100n; footprint Capacitor_SMD:C_0805_2012Metric_Pad1.15x1.40mm_HandSolder -> Capacitor_SMD:C_0402_1005Metric; moved to F.Cu
- D0, D1, D10, D11, D12, D13, D14, D15, D16, D17, D18, D19, D2, D20, D21, D22, D23, D24, D25, D26, D27, D28, D29, D3, D30, D31, D32, D33, D34, D35, D36, D37, D38, D39, D4, D40, D41, D42, D43, D44, D45, D46, D47, D48, D49, D5, D50, D51, D52, D53, D54, D55, D56, D57, D58, D59, D6, D60, D61, D62, D63, D64, D65, D66, D7, D8, D9: value D -> 1N4148WS; footprint Diode_SMD:D_0805_2012Metric_Pad1.15x1.40mm_HandSolder -> Diode_SMD:D_SOD-323_HandSoldering
- J1: value USB_mini_micro_B -> USB_C_Receptacle_USB2.0_16P; footprint Connector_USB:USB_Mini-B_Wuerth_65100516121_Horizontal -> Connector_USB:USB_C_Receptacle_G-Switch_GT-USB-7010ASV; moved to F.Cu
- K33: value D -> KeyD
- K47: value C -> KeyD
- R1: value 10k -> 1k; footprint Resistor_SMD:R_0805_2012Metric_Pad1.15x1.40mm_HandSolder -> Resistor_SMD:R_0402_1005Metric; moved to F.Cu
- R2, R3: value 22R -> 27; footprint Resistor_SMD:R_0805_2012Metric_Pad1.15x1.40mm_HandSolder -> Resistor_SMD:R_0402_1005Metric; moved to F.Cu
- R4: footprint Resistor_SMD:R_0805_2012Metric_Pad1.15x1.40mm_HandSolder -> Resistor_SMD:R_0603_1608Metric; moved to F.Cu
- SW1: footprint Button_Switch_SMD:SW_Push_1P1T_NO_6x6mm_H9.5mm -> Button_Switch_SMD:SW_Push_1P1T_NO_CK_KMR2; moved to F.Cu
- U1: value ATmega32U4-AU -> RP2040; footprint Package_QFP:TQFP-44_10x10mm_P0.8mm -> Package_DFN_QFN:QFN-56-1EP_7x7mm_P0.4mm_EP3.2x3.2mm; moved to F.Cu
- Y1: value Crystal -> ABM8-272-T3; footprint Crystal:Crystal_SMD_5032-2Pin_5.0x3.2mm_HandSoldering -> parts:ABM8272T3; moved to F.Cu
- moved H1 194.3 mm to (65.0, 87.6)
- moved D35 182.7 mm to (175.2, 158.9)
- moved D37 182.7 mm to (213.3, 158.9)
- moved D40 182.7 mm to (270.4, 158.9)
- moved D41 182.7 mm to (289.5, 158.9)
- moved K47 182.7 mm to (152.4, 169.0)
- moved K55 182.7 mm to (311.9, 169.0)
- moved D0 182.7 mm to (65.6, 120.8)
- moved D1 182.7 mm to (84.7, 120.8)
- moved D12 182.7 mm to (294.2, 120.8)
- moved D13 182.7 mm to (322.8, 120.8)
- moved D15 182.7 mm to (70.4, 139.8)
- moved D16 182.7 mm to (94.2, 139.8)
- moved D17 182.7 mm to (113.3, 139.8)
- moved D18 182.7 mm to (132.3, 139.8)
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Connections:
- C1 pad 1: VCC -> Net-(U1-XIN)
- C2 pad 1: VCC -> Net-(C2-Pad1)
- C3 pad 1: VCC -> +1V1
- C4 pad 1: VCC -> +1V1
- C5 pad 1: VCC -> +1V1
- C6 pad 1: Net-(C6-Pad1) -> +3V3
- C7 pad 1: Net-(C7-Pad1) -> +3V3
- C8 pad 1: Net-(C8-Pad1) -> +3V3
- K43 pad 1: /Col_13 -> /Col_14
- K57 pad 1: /Col_13 -> /Col_14
- K61 pad 1: /Col_3 -> /Col_5
- K62 pad 1: /Col_4 -> /Col_9
- K63 pad 1: /Col_5 -> /Col_10
- K64 pad 1: /Col_6 -> /Col_11
- K65 pad 1: /Col_7 -> /Col_12
- K66 pad 1: /Col_8 -> /Col_14
- R1 pad 1: Net-(R1-Pad1) -> Net-(U1-XOUT)
- R1 pad 2: VCC -> Net-(C2-Pad1)
- R2 pad 1: Net-(R2-Pad1) -> Net-(U1-USB_DP)
- R2 pad 2: Net-(J1-Pad2) -> /USB_D+
- R3 pad 1: Net-(R3-Pad1) -> Net-(U1-USB_DM)
- R3 pad 2: Net-(J1-Pad3) -> /USB_D-
- R4 pad 1: GND -> /RUN
- R4 pad 2: Net-(R4-Pad2) -> +3V3
- SW1 pad 2: Net-(R1-Pad1) -> /RUN
- U1 pad 1: /Row_6 -> +3V3
- U1 pad 10: /Row_3 -> +3V3
- U1 pad 11: /Row_2 -> /Col_3
- U1 pad 12: /Row_1 -> /Col_4
- U1 pad 13: Net-(R1-Pad1) -> /Col_5
- U1 pad 14: VCC -> /Col_6
- U1 pad 15: GND -> /Col_7
- U1 pad 16: Net-(C7-Pad1) -> /Col_8
- U1 pad 17: Net-(C6-Pad1) -> /Col_9
- U1 pad 18: /Row_0 -> /Col_10
- U1 pad 19: /Col_15 -> GND
- U1 pad 2: VCC -> /Row_0
- U1 pad 20: /Col_16 -> Net-(U1-XIN)
- U1 pad 21: /Col_17 -> Net-(U1-XOUT)
- U1 pad 22: /Col_14 -> +3V3
- U1 pad 23: GND -> +1V1
- U1 pad 24: VCC -> /SWCLK
- U1 pad 25: /Col_7 -> /SWD
- U1 pad 26: /Col_6 -> /RUN
- U1 pad 27: /Col_5 -> /Col_11
- U1 pad 28: /Col_4 -> /Col_12
- U1 pad 29: /Col_3 -> /Col_13
- U1 pad 3: Net-(R3-Pad1) -> /Row_1
- U1 pad 30: /Col_2 -> /Col_14
- U1 pad 31: /Col_1 -> unconnected-(U1-GPIO20-Pad31)
- U1 pad 32: /Col_0 -> unconnected-(U1-GPIO21-Pad32)
- U1 pad 33: Net-(R4-Pad2) -> +3V3
- U1 pad 34: VCC -> unconnected-(U1-GPIO22-Pad34)
- U1 pad 35: GND -> unconnected-(U1-GPIO23-Pad35)
- U1 pad 36: /Col_8 -> unconnected-(U1-GPIO24-Pad36)
- U1 pad 37: /Col_9 -> unconnected-(U1-GPIO25-Pad37)
- U1 pad 38: /Col_10 -> unconnected-(U1-GPIO26_ADC0-Pad38)
- U1 pad 39: /Col_11 -> unconnected-(U1-GPIO27_ADC1-Pad39)
- U1 pad 4: Net-(R2-Pad1) -> /Row_2
- U1 pad 40: /Col_12 -> unconnected-(U1-GPIO28_ADC2-Pad40)
- U1 pad 41: /Col_13 -> unconnected-(U1-GPIO29_ADC3-Pad41)
- U1 pad 42: Net-(U1-Pad42) -> +3V3
- U1 pad 43: GND -> +3V3
- U1 pad 44: VCC -> +3V3
- U1 pad 5: GND -> /Row_3
- U1 pad 6: Net-(C8-Pad1) -> /Row_4
- U1 pad 7: VCC -> /Col_0
- U1 pad 8: /Row_5 -> /Col_1
- U1 pad 9: /Row_4 -> /Col_2
- Y1 pad 1: Net-(C6-Pad1) -> Net-(U1-XIN)
- Y1 pad 2: Net-(C7-Pad1) -> GND
Routing:
- net /Col_0: track 84.1 -> 367.8 mm
- net /Col_1: track 98.0 -> 357.1 mm
- net /Col_2: track 98.0 -> 337.9 mm
- net +3V3: track 0.00 -> 232.5 mm, vias 0 -> 21
- net /Col_3: track 102.3 -> 292.9 mm
- net /Col_5: track 102.3 -> 275.5 mm
- net /Col_4: track 102.3 -> 273.8 mm
- net /Row_4: track 281.0 -> 430.0 mm, vias 0 -> 1
- net /Col_6: track 102.3 -> 235.3 mm
- net /Row_3: track 273.8 -> 405.5 mm, vias 0 -> 1
- net /Col_9: track 71.1 -> 200.8 mm
- net /Row_2: track 278.6 -> 393.7 mm, vias 0 -> 1
- net /Col_7: track 102.3 -> 217.0 mm
- net /Col_10: track 71.1 -> 184.2 mm
- net /Col_11: track 75.5 -> 176.2 mm
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- added copper zone on F.Cu, net +1V1
- added copper zone on F.Cu, net +3V3
- added copper zone on B.Cu, net GND
Other:
- board outline added: 308 x 123.8 mm
- net class Default removed
- rule pad_to_mask_clearance: 0.051 -> 0.038
- rule solder_mask_min_width: 0.25 -> 0.1

Commit message: more random ahh changes
Parts:
- removed the ? at (350.5, 92.5)
- removed the ? at (349.2, 92.5)
- removed the ? at (351.8, 92.5)
- removed the ? at (350.5, 91.3)
- removed the ? at (350.5, 93.8)
- removed R10, R11, R12, R13, R14, R15, R16, R17, R18, R19, R20, R21, R22, R8, R9: 10k, Resistor_SMD:R_0603_1608Metric
- ? (x4), J1, SW1, SW2, U1, U2, Y1: moved to B.Cu
- C1, C2: value 16pF -> 0402CG150J500NT; moved to B.Cu
- C10, C11, C12, C13, C3, C4, C7, C8, C9: value 100n -> CL05B104KO5NNNC; moved to B.Cu
- C14, C16: value 10uF -> CL05A106MQ5NUNC; footprint Capacitor_SMD:C_0805_2012Metric -> Capacitor_SMD:C_0402_1005Metric; moved to B.Cu
- C15: value 0.1uf -> CL05A105KA5NQNC; footprint Capacitor_SMD:C_0603_1608Metric -> Capacitor_SMD:C_0402_1005Metric; moved to B.Cu
- C5, C6: value 1u -> CL05A105KA5NQNC; moved to B.Cu
- R1: value 1k -> 0402WGF1001TCE; moved to B.Cu
- R2, R3: value 27 -> RTT0527R4FTP; footprint Resistor_SMD:R_0402_1005Metric -> Resistor_SMD:R_0805_2012Metric; moved to B.Cu
- R4: value 10k -> 0402WGF1001TCE; footprint Resistor_SMD:R_0603_1608Metric -> Resistor_SMD:R_0402_1005Metric; moved to B.Cu
- R5, R6: value 5.1k -> 0402WGF5101TCE; footprint Resistor_SMD:R_0603_1608Metric -> Resistor_SMD:R_0402_1005Metric; moved to B.Cu
- R7: value 1k -> 0402WGF1001TCE; footprint Resistor_SMD:R_0603_1608Metric -> Resistor_SMD:R_0402_1005Metric; moved to B.Cu
- U3: value NCP1117-3.3_SOT223 -> AMS1117-3.3; moved to B.Cu
- moved C16 73.2 mm to (359.6, 100.4), turned to 90 degrees
- moved C14 66.3 mm to (363.2, 93.6)
- moved U3 63.0 mm to (354.0, 100.9), turned to 180 degrees
- moved J1 57.7 mm to (358.9, 85.6), turned to 0 degrees
- moved R6 49.8 mm to (354.8, 94.0), turned to 180 degrees
- moved R5 49.8 mm to (354.8, 92.9), turned to 180 degrees
- moved H2 35.7 mm to (312.3, 86.2)
- moved C8 35.5 mm to (322.6, 93.4), turned to 180 degrees
- moved SW3 34.9 mm to (76.4, 100.5), turned to 90 degrees
- moved C6 31.9 mm to (323.7, 89.4), turned to 180 degrees
- moved C7 31.9 mm to (323.7, 88.3), turned to 180 degrees
- moved R4 30.0 mm to (347.1, 96.9)
- moved R3 29.9 mm to (324.3, 84.7)
- moved SW1 27.1 mm to (345.8, 93.3)
- moved R2 27.0 mm to (326.2, 84.7)
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Connections:
- R4 pad 1: /RUN -> +3V3
- R4 pad 2: +3V3 -> /RUN
- SW3 pad A: unconnected-(SW3-PadA) -> /SW3_A
- SW3 pad B: unconnected-(SW3-PadB) -> /SW3_B
- SW3 pad C: unconnected-(SW3-PadC) -> GND
- SW3 pad MP: unconnected-(SW3-PadMP) -> GND
- SW3 pad S1: unconnected-(SW3-PadS1) -> /SW3_Button
- SW3 pad S2: unconnected-(SW3-PadS2) -> GND
- SW4 pad A: unconnected-(SW4-PadA) -> /SW4_A
- SW4 pad B: unconnected-(SW4-PadB) -> /SW4_B
- SW4 pad C: unconnected-(SW4-PadC) -> GND
- SW4 pad MP: unconnected-(SW4-PadMP) -> GND
- SW4 pad S1: unconnected-(SW4-PadS1) -> /SW4_Button
- SW4 pad S2: unconnected-(SW4-PadS2) -> GND
- U1 pad 11: /Col_3 -> /Col_11
- U1 pad 12: /Col_4 -> /Col_10
- U1 pad 13: /Col_5 -> /Col_9
- U1 pad 14: /Col_6 -> /Col_8
- U1 pad 16: /Col_8 -> /Col_6
- U1 pad 17: /Col_9 -> /Col_5
- U1 pad 18: /Col_10 -> /Col_4
- U1 pad 27: /Col_11 -> /Col_3
- U1 pad 28: /Col_12 -> /Col_2
- U1 pad 29: /Col_13 -> /Col_1
- U1 pad 30: /Col_14 -> /Col_0
- U1 pad 31: unconnected-(U1-GPIO20-Pad31) -> /SW4_B
- U1 pad 32: unconnected-(U1-GPIO21-Pad32) -> /SW4_A
- U1 pad 34: unconnected-(U1-GPIO22-Pad34) -> /SW4_Button
- U1 pad 35: unconnected-(U1-GPIO23-Pad35) -> /SW3_B
- U1 pad 36: unconnected-(U1-GPIO24-Pad36) -> /SW3_A
- U1 pad 37: unconnected-(U1-GPIO25-Pad37) -> /SW3_Button
- U1 pad 7: /Col_0 -> /Col_14
- U1 pad 8: /Col_1 -> /Col_13
- U1 pad 9: /Col_2 -> /Col_12
Routing:
- net /SW3_Button: track 0.00 -> 253.8 mm, vias 0 -> 1
- net /SW3_A: track 0.00 -> 252.6 mm
- net /SW3_B: track 0.00 -> 247.5 mm
- net /SW4_A: track 0.00 -> 234.1 mm
- net /SW4_B: track 0.00 -> 228.9 mm
- net /SW4_Button: track 0.00 -> 228.0 mm, vias 0 -> 1
- net GND: track 51.7 -> 264.7 mm, vias 12 -> 15
- net +3V3: track 232.5 -> 78.9 mm, vias 21 -> 11
- net /Row_0: track 366.4 -> 333.2 mm, vias 1 -> 2
- net /Row_1: track 380.0 -> 347.2 mm, vias 1 -> 2
- net /Row_2: track 393.7 -> 364.5 mm, vias 1 -> 2
- net /Row_3: track 405.5 -> 377.5 mm, vias 1 -> 2
- net /Row_4: track 430.0 -> 403.1 mm, vias 1 -> 2
- net /Col_2: track 337.9 -> 316.4 mm
- net /Col_1: track 357.1 -> 335.7 mm
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- added copper zone on B.Cu, net +1V1
- added copper zone on B.Cu, net +3V3
- added copper zone on F.Cu, net GND
- removed copper zone on F.Cu, net +1V1
- removed copper zone on F.Cu, net +3V3
- removed copper zone on B.Cu, net GND

Commit message: stuff
Parts:
- C1, C2: value 0402CG150J500NT -> 0402CG200J500NT
- SW1, SW2: footprint Button_Switch_SMD:SW_Push_1P1T_NO_CK_KMR2 -> Button_Switch_THT:SW_PUSH_1P1T_6x3.5mm_H4.3_APEM_MJTP1243; moved to F.Cu
- moved H1 6.68 mm to (63.7, 92.6)
- moved R4 5.59 mm to (341.6, 97.6)
- moved SW1 5.11 mm to (341.0, 95.1)
- moved H2 4.80 mm to (309.1, 89.8)
- moved SW2 4.76 mm to (346.2, 95.1)
- moved SW4 3.33 mm to (98.5, 102.0)
- moved ? 3.06 mm to (328.7, 93.4)
- moved C1 3.06 mm to (324.9, 104.5)
- moved C10 3.06 mm to (325.4, 102.0)
- moved C12 3.06 mm to (333.1, 91.3)
- moved C2 3.06 mm to (324.9, 103.5)
- moved C4 3.06 mm to (328.9, 87.8)
- moved C7 3.06 mm to (322.3, 91.1)
- moved R1 3.06 mm to (327.7, 99.8)
- moved R6 3.06 mm to (353.4, 96.7)
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Connections:
- SW1 pad 1: GND -> /RUN
- SW1 pad 2: /RUN -> GND
Routing:
- net GND: track 264.7 -> 252.4 mm, vias 15 -> 13
- net /~{BOOTSEL}: track 17.7 -> 7.44 mm
- net /RUN: track 27.5 -> 20.3 mm, vias 2 -> 1
- net /SW4_A: track 234.1 -> 227.9 mm
- net /SW4_B: track 228.9 -> 222.7 mm
- net /SW3_Button: track 253.8 -> 248.1 mm
- net /SW4_Button: track 228.0 -> 224.9 mm
- net /Col_0: track 346.5 -> 344.0 mm
- net /Col_1: track 335.7 -> 333.1 mm
- net /Col_9: track 194.2 -> 191.7 mm
- net /Col_8: track 191.0 -> 188.4 mm
- net /Col_5: track 267.6 -> 265.1 mm
- net /Col_11: track 162.1 -> 159.6 mm
- net /Col_10: track 178.2 -> 175.6 mm
- net /Col_6: track 227.9 -> 225.4 mm
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Other:
- board size 308 x 123.8 mm -> 308 x 121.3 mm

Commit message: move part nums to description
Parts:
- C1, C2: value 0402CG200J500NT -> 20pF±5%
- C10, C11, C12, C13, C3, C4, C7, C8, C9: value CL05B104KO5NNNC -> 0.1 µF ±10%
- C14, C16: value CL05A106MQ5NUNC -> 10 µF ±20%
- C15, C5, C6: value CL05A105KA5NQNC -> 1 µF ±10%
- R1, R4, R7: value 0402WGF1001TCE -> 1k
- R5, R6: value 0402WGF5101TCE -> 5.1k
Changed lines of the file:
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@@
 			)
 		)
-		(property "Value" "0402WGF1001TCE"
+		(property "Value" "1k"
 			(at 0 -1.17 0)
 			(layer "B.Fab")
@@
 			)
 		)
-		(property "Datasheet" ""
+		(property "Datasheet" "https://www.mouser.com/datasheet/2/1365/1-3044649.pdf"
 			(at 0 0 0)
 			(unlocked yes)
@@
 			)
 		)
-		(property "Description" ""
+		(property "Description" "0402WGF1001TCE"
 			(at 0 0 0)
 			(unlocked yes)
@@
 			)
 		)
-		(property "Value" "CL05A106MQ5NUNC"
+		(property "Value" "10 µF ±20%"
 			(at 0 -1.16 -90)
 			(layer "B.Fab")
@@
 			)
 		)
-		(property "Datasheet" ""
+		(property "Datasheet" "https://mm.digikey.com/Volume0/opasdata/d220001/medias/docus/41/CL05A106MQ5NUNC_Spec.pdf"
 			(at 0 0 -90)
 			(unlocked yes)
@@
 			)
 		)
-		(property "Description" ""
+		(property "Description" "CL05A106MQ5NUNC"
 			(at 0 0 -90)
 			(unlocked yes)
@@
 			)
 		)
-		(property "Value" "CL05A106MQ5NUNC"
+		(property "Value" "10 µF ±20%"
 			(at 0 -1.16 -90)
 			(layer "B.Fab")
@@
 			)
 		)
-		(property "Datasheet" ""
+		(property "Datasheet" "https://mm.digikey.com/Volume0/opasdata/d220001/medias/docus/41/CL05A106MQ5NUNC_Spec.pdf"
 			(at 0 0 -90)
 			(unlocked yes)
@@
 			)
 		)
-		(property "Description" ""
+		(property "Description" "CL05A106MQ5NUNC"
 			(at 0 0 -90)
 			(unlocked yes)
@@
 			)
 		)
-		(property "Value" "CL05B104KO5NNNC"
+		(property "Value" "0.1 µF ±10%"
 			(at 0 -1.16 135)
 			(layer "B.Fab")
@@
 			)
 		)
-		(property "Datasheet" ""
+		(property "Datasheet" "https://mm.digikey.com/Volume0/opasdata/d220001/medias/docus/609/CL05B104KO5NNNC.pdf"
 			(at 0 0 -45)
 			(unlocked yes)
@@
 			)
 		)
-		(property "Description" ""
+		(property "Description" "CL05B104KO5NNNC"
 			(at 0 0 -45)
 			(unlocked yes)
@@
 			)
 		)
-		(property "Value" "CL05B104KO5NNNC"
+		(property "Value" "0.1 µF ±10%"
 			(at 0 -1.16 90)
 			(layer "B.Fab")
@@
 			)
 		)
-		(property "Datasheet" ""
+		(property "Datasheet" "https://mm.digikey.com/Volume0/opasdata/d220001/medias/docus/609/CL05B104KO5NNNC.pdf"
 			(at 0 0 -90)
 			(unlocked yes)
@@
 			)
 		)
-		(property "Description" ""
+		(property "Description" "CL05B104KO5NNNC"
 			(at 0 0 -90)
 			(unlocked yes)
@@
 			)
 		)
-		(property "Value" "CL05B104KO5NNNC"
+		(property "Value" "0.1 µF ±10%"
 			(at 0 -1.16 0)
 			(layer "B.Fab")
@@
 			)
 		)
-		(property "Datasheet" ""
+		(property "Datasheet" "https://mm.digikey.com/Volume0/opasdata/d220001/medias/docus/609/CL05B104KO5NNNC.pdf"
 			(at 0 0 0)
 			(unlocked yes)
@@
 			)
 		)
-		(property "Description" ""
+		(property "Description" "CL05B104KO5NNNC"
 			(at 0 0 0)
 			(unlocked yes)
@@
 			)
 		)
-		(property "Value" "CL05B104KO5NNNC"
+		(property "Value" "0.1 µF ±10%"
 			(at 0 -1.16 90)
 			(layer "B.Fab")
@@
 			)
 		)
-		(property "Datasheet" ""
+		(property "Datasheet" "https://mm.digikey.com/Volume0/opasdata/d220001/medias/docus/609/CL05B104KO5NNNC.pdf"
 			(at 0 0 -90)
 			(unlocked yes)
@@
 			)
 		)
-		(property "Description" ""
+		(property "Description" "CL05B104KO5NNNC"
 			(at 0 0 -90)
 			(unlocked yes)
@@
 			)
 		)
-		(property "Value" "CL05A105KA5NQNC"
+		(property "Value" "1 µF ±10%"
 			(at 0 -1.16 -90)
 			(layer "B.Fab")
@@
 			)
 		)
-		(property "Datasheet" ""
+		(property "Datasheet" "https://mm.digikey.com/Volume0/opasdata/d220001/medias/docus/41/CL05A105KA5NQNC.pdf"
 			(at 0 0 -90)
 			(unlocked yes)
@@
 			)
 		)
-		(property "Description" ""
+		(property "Description" "CL05A105KA5NQNC"
 			(at 0 0 -90)
 			(unlocked yes)
@@
 			)
 		)
-		(property "Value" "0402WGF1001TCE"
+		(property "Value" "1k"
 			(at 0 -1.17 -90)
 			(layer "B.Fab")
@@
 			)
 		)
-		(property "Datasheet" ""
+		(property "Datasheet" "https://www.mouser.com/datasheet/2/1365/1-3044649.pdf"
 			(at 0 0 -90)
 			(unlocked yes)
@@
 			)
 		)
-		(property "Description" ""
+		(property "Description" "0402WGF1001TCE"
 			(at 0 0 -90)
 			(unlocked yes)
@@
 			)
 		)
-		(property "Value" "0402CG200J500NT"
+		(property "Value" "20pF±5%"
 			(at 0 -1.16 0)
 			(layer "B.Fab")
@@
 			)
 		)
-		(property "Datasheet" ""
+		(property "Datasheet" "https://www.lcsc.com/datasheet/lcsc_datasheet_2304140030_FH--Guangdong-Fenghua-Advanced-Tech-0402CG200J500NT_C1554.pdf"
 			(at 0 0 0)
 			(unlocked yes)
@@
 			)
 		)
-		(property "Description" ""
+		(property "Description" "0402CG200J500NT"
 			(at 0 0 0)
 			(unlocked yes)
@@
 			)
 		)
-		(property "Value" "CL05B104KO5NNNC"
+		(property "Value" "0.1 µF ±10%"
 			(at 0 -1.16 90)
 			(layer "B.Fab")
@@
 			)
 		)
-		(property "Datasheet" ""
+		(property "Datasheet" "https://mm.digikey.com/Volume0/opasdata/d220001/medias/docus/609/CL05B104KO5NNNC.pdf"
 			(at 0 0 -90)
 			(unlocked yes)
@@
 			)
 		)
-		(property "Description" ""
+		(property "Description" "CL05B104KO5NNNC"
 			(at 0 0 -90)
 			(unlocked yes)
@@
 			)
 		)
-		(property "Value" "CL05A105KA5NQNC"
+		(property "Value" "1 µF ±10%"
 			(at 0 -1.16 90)
 			(layer "B.Fab")
@@
 			)
 		)
-		(property "Datasheet" ""
+		(property "Datasheet" "https://mm.digikey.com/Volume0/opasdata/d220001/medias/docus/41/CL05A105KA5NQNC.pdf"
 			(at 0 0 90)
 			(unlocked yes)
@@
 			)
 		)
-		(property "Description" ""
+		(property "Description" "CL05A105KA5NQNC"
 			(at 0 0 90)
 			(unlocked yes)
@@
 			)
 		)
-		(property "Value" "CL05B104KO5NNNC"
+		(property "Value" "0.1 µF ±10%"
 			(at 0 -1.16 90)
 			(layer "B.Fab")
@@
 			)
 		)
-		(property "Datasheet" ""
+		(property "Datasheet" "https://mm.digikey.com/Volume0/opasdata/d220001/medias/docus/609/CL05B104KO5NNNC.pdf"
 			(at 0 0 90)
 			(unlocked yes)
@@
 			)
 		)
-		(property "Description" ""
+		(property "Description" "CL05B104KO5NNNC"
 			(at 0 0 90)
 			(unlocked yes)
@@
 			)
 		)
-		(property "Value" "0402WGF1001TCE"
+		(property "Value" "1k"
 			(at 0 -1.17 0)
 			(layer "B.Fab")
@@
 			)
 		)
-		(property "Datasheet" ""
+		(property "Datasheet" "https://www.mouser.com/datasheet/2/1365/1-3044649.pdf"
 			(at 0 0 0)
 			(unlocked yes)
@@
 			)
 		)
-		(property "Description" ""
+		(property "Description" "0402WGF1001TCE"
 			(at 0 0 0)
 			(unlocked yes)
@@
 			)
 		)
-		(property "Value" "0402CG200J500NT"
+		(property "Value" "20pF±5%"
 			(at 0 -1.16 0)
 			(layer "B.Fab")
@@
 			)
 		)
-		(property "Datasheet" ""
+		(property "Datasheet" "https://www.lcsc.com/datasheet/lcsc_datasheet_2304140030_FH--Guangdong-Fenghua-Advanced-Tech-0402CG200J500NT_C1554.pdf"
 			(at 0 0 0)
 			(unlocked yes)
@@
 			)
 		)
-		(property "Description" ""
+		(property "Description" "0402CG200J500NT"
 			(at 0 0 0)
 			(unlocked yes)
@@
 			)
 		)
-		(property "Value" "CL05B104KO5NNNC"
+		(property "Value" "0.1 µF ±10%"
 			(at 0 -1.16 90)
 			(layer "B.Fab")
@@
 			)
 		)
-		(property "Datasheet" ""
+		(property "Datasheet" "https://mm.digikey.com/Volume0/opasdata/d220001/medias/docus/609/CL05B104KO5NNNC.pdf"
 			(at 0 0 90)
 			(unlocked yes)
@@
 			)
 		)
-		(property "Description" ""
+		(property "Description" "CL05B104KO5NNNC"
 			(at 0 0 90)
 			(unlocked yes)
@@
 			)
 		)
-		(property "Value" "0402WGF5101TCE"
+		(property "Value" "5.1k"
 			(at 0 -1.17 0)
 			(layer "B.Fab")
@@
 			)
 		)
-		(property "Datasheet" ""
+		(property "Datasheet" "https://wmsc.lcsc.com/wmsc/upload/file/pdf/v2/lcsc/2206010045_UNI-ROYAL-Uniroyal-Elec-0402WGF5101TCE_C25905.pdf"
 			(at 0 0 0)
 			(unlocked yes)
@@
 			)
 		)
-		(property "Description" "Resistor"
+		(property "Description" "0402WGF5101TCE"
 			(at 0 0 0)
 			(unlocked yes)
@@
 			)
 		)
-		(property "Value" "CL05B104KO5NNNC"
+		(property "Value" "0.1 µF ±10%"
 			(at 0 -1.16 0)
 			(layer "B.Fab")
@@
 			)
 		)
-		(property "Datasheet" ""
+		(property "Datasheet" "https://mm.digikey.com/Volume0/opasdata/d220001/medias/docus/609/CL05B104KO5NNNC.pdf"
 			(at 0 0 0)
 			(unlocked yes)
@@
 			)
 		)
-		(property "Description" ""
+		(property "Description" "CL05B104KO5NNNC"
 			(at 0 0 0)
 			(unlocked yes)
@@
 			)
 		)
-		(property "Value" "CL05A105KA5NQNC"
+		(property "Value" "1 µF ±10%"
 			(at 0 -1.16 0)
 			(layer "B.Fab")
@@
 			)
 		)
-		(property "Datasheet" ""
+		(property "Datasheet" "https://mm.digikey.com/Volume0/opasdata/d220001/medias/docus/41/CL05A105KA5NQNC.pdf"
 			(at 0 0 0)
 			(unlocked yes)
@@
 			)
 		)
-		(property "Description" ""
+		(property "Description" "CL05A105KA5NQNC"
 			(at 0 0 0)
 			(unlocked yes)
@@
 			)
 		)
-		(property "Value" "0402WGF5101TCE"
+		(property "Value" "5.1k"
 			(at 0 -1.17 0)
 			(layer "B.Fab")
@@
 			)
 		)
-		(property "Datasheet" ""
+		(property "Datasheet" "https://wmsc.lcsc.com/wmsc/upload/file/pdf/v2/lcsc/2206010045_UNI-ROYAL-Uniroyal-Elec-0402WGF5101TCE_C25905.pdf"
 			(at 0 0 0)
 			(unlocked yes)
@@
 			)
 		)
-		(property "Description" "Resistor"
+		(property "Description" "0402WGF5101TCE"
 			(at 0 0 0)
 			(unlocked yes)
@@
 			)
 		)
-		(property "Value" "CL05B104KO5NNNC"
+		(property "Value" "0.1 µF ±10%"
 			(at 0 -1.16 135)
 			(layer "B.Fab")
@@
 			)
 		)
-		(property "Datasheet" ""
+		(property "Datasheet" "https://mm.digikey.com/Volume0/opasdata/d220001/medias/docus/609/CL05B104KO5NNNC.pdf"
 			(at 0 0 -45)
 			(unlocked yes)
@@
 			)
 		)
-		(property "Description" ""
+		(property "Description" "CL05B104KO5NNNC"
 			(at 0 0 -45)
 			(unlocked yes)
