File: mykb/mykb.kicad_sch (KiCad schematic)
At the start: 183 parts, among them J2 USB_C_Receptacle_USB2.0_16P, K0 Esc, K1 !,1, K10 ),0, K11 _,-, K12 +,=, K13 Backspace, K14 Home, K15 Tab, K16 Q, K17 W, K18 E, K19 R, K2 @,2, K20 T, K21 Y, K22 U, K23 I, K24 O, K25 P, K26 {,[, K27 },], K28 |,\, K29 PgUp, K3 #,3, K30 Caps Lock, K31 A, K32 S, K33 Key_D, K34 F, K35 G, K36 H, K37 J, K38 K, K39 L, K4 $,4, K40 :,;, K41 ",', K42 Enter, K43 PgDn, K44 Shift, K45 Z, K46 X, K47 C, K48 V, K49 B, K5 %,5, K50 N, K51 M, K52 <,,, K53 >,., K54 ?,/, K55 Shift, K56 ↑, K57 End, K58 Ctrl, K59 Cmd, K6 ^,6, K60 Alt, K61 Blank, K62 Alt, K63 Ctrl, K64 ←, K65 ↓, K66 →, K7 &,7, K8 *,8, K9 (,9, SW1 SW_Push, SW2 SW_Push, U1 RP2040, U2 NCP1117-3.3_SOT223, U4 W25Q128JVS, Y1 Crystal_GND24

Commit message: progress on the redo
Parts:
- removed J2: USB_C_Receptacle_USB2.0_16P, Connector_USB:USB_C_Receptacle_G-Switch_GT-USB-7010ASV, symbol Connector:USB_C_Receptacle_USB2.0_16P
- removed U2: NCP1117-3.3_SOT223, Package_TO_SOT_SMD:SOT-223-3_TabPin2, symbol Regulator_Linear:NCP1117-3.3_SOT223
- removed U4: W25Q128JVS, Package_SO:SOIC-8_5.23x5.23mm_P1.27mm, symbol Memory_Flash:W25Q128JVS
- added J1: USB_C_Receptacle_USB2.0_16P, Connector_USB:USB_C_Receptacle_G-Switch_GT-USB-7010ASV, symbol Connector:USB_C_Receptacle_USB2.0_16P
- added SW3, SW4: RotaryEncoder_Switch_MP, Rotary_Encoder:RotaryEncoder_Alps_EC11E-Switch_Vertical_H20mm, symbol Device:RotaryEncoder_Switch_MP
- added U2: W25Q128JVS, Package_SO:SOIC-8_5.23x5.23mm_P1.27mm, symbol Memory_Flash:W25Q128JVS
- added U3: NCP1117-3.3_SOT223, Package_TO_SOT_SMD:SOT-223-3_TabPin2, symbol Regulator_Linear:NCP1117-3.3_SOT223
- C1, C10, C11, C12, C13, C2, C9: footprint Capacitor_SMD:C_0603_1608Metric -> Capacitor_SMD:C_0402_1005Metric
- C14: value 100n -> 10uF; footprint Capacitor_SMD:C_0603_1608Metric -> Capacitor_SMD:C_0805_2012Metric
- C15: value 100n -> 0.1uf
- C16: value 0.1uf -> 10uF; footprint Capacitor_SMD:C_0603_1608Metric -> Capacitor_SMD:C_0805_2012Metric
- C3, C4: value 10uF -> 100n; footprint Capacitor_SMD:C_0805_2012Metric -> Capacitor_SMD:C_0402_1005Metric
- C5: value 100n -> 1u
- C8: value 1u -> 100n
- K33: value Key_D -> KeyD
- K47: value C -> KeyD
- R1: footprint Resistor_SMD:R_0603_1608Metric -> Resistor_SMD:R_0402_1005Metric
- R10, R11, R13, R14, R15, R16, R17, R18, R19, R20, R21, R22, R8, R9: footprint Resistor_THT:R_Axial_DIN0309_L9.0mm_D3.2mm_P15.24mm_Horizontal -> Resistor_SMD:R_0603_1608Metric
- R4: value 1k -> 10k
- R7: value 10k -> 1k; footprint Resistor_THT:R_Axial_DIN0309_L9.0mm_D3.2mm_P15.24mm_Horizontal -> Resistor_SMD:R_0603_1608Metric
- Y1: value Crystal_GND24 -> ABM8-272-T3
Connections:
- net +1V1: now also C3.1, C4.1; no longer C6.1, C7.1
- net +3V3: now also C6.1, C7.1, R4.2, U2.8 (VCC), U3.2 (VO); no longer C14.1, C4.1, R7.2
- net +5V: now also C14.1, J1.A4 (VBUS), J1.A9 (VBUS), J1.B4 (VBUS), J1.B9 (VBUS), U3.3 (VI); no longer C3.1
- net Col_0: now also R8.1; no longer R7.1
- net Col_1: now also R9.1; no longer R8.1
- net Col_13: no longer K43.1, K57.1, K66.1
- net Col_14: now also K43.1, K57.1, K66.1
- net Col_2: now also R10.1; no longer R9.1
- net Col_3: now also R11.1; no longer R10.1
- net Col_4: now also R12.1; no longer R11.1
- net GND: now also J1.A1 (GND), J1.A12 (GND), J1.B1 (GND), J1.B12 (GND), J1.S1 (SHIELD), U2.4 (GND), U3.1 (GND)
- net QSPI_SCLK: now also U2.6 (CLK)
- net QSPI_SD0: now also U2.5 (DI(IO0))
- net QSPI_SD1: now also U2.2 (DO(IO1))
- net QSPI_SD2: now also U2.3 (IO2)
- net QSPI_SD3: now also U2.7 (IO3)
- net QSPI_SS: now also R7.1, U2.1 (~{CS}); no longer R4.1
- net RUN: now also R4.1; no longer R12.1
- net USB_D+: now also J1.A6 (D+), J1.B6 (D+)
- net USB_D-: now also J1.A7 (D-), J1.B7 (D-)
- net ~{BOOTSEL}: now also R7.2; no longer R4.2
- net at R6.1: now also J1.B5 (CC2)
- net at R5.1: now also J1.A5 (CC1)
Other:
- moved on the sheet: H1, H2, H3, H4

Commit message: more random ahh changes
Parts:
- removed R10, R11, R12, R13, R14, R15, R16, R17, R18, R19, R20, R21, R22, R8, R9: 10k, Resistor_SMD:R_0603_1608Metric, symbol Device:R
- C1, C2: value 16pF -> 0402CG150J500NT
- C10, C11, C12, C13, C3, C4, C7, C8, C9: value 100n -> CL05B104KO5NNNC
- C14, C16: value 10uF -> CL05A106MQ5NUNC; footprint Capacitor_SMD:C_0805_2012Metric -> Capacitor_SMD:C_0402_1005Metric
- C15: value 0.1uf -> CL05A105KA5NQNC; footprint Capacitor_SMD:C_0603_1608Metric -> Capacitor_SMD:C_0402_1005Metric
- C5, C6: value 1u -> CL05A105KA5NQNC
- R1: value 1k -> 0402WGF1001TCE
- R2, R3: value 27 -> RTT0527R4FTP; footprint Resistor_SMD:R_0402_1005Metric -> Resistor_SMD:R_0805_2012Metric
- R4: value 10k -> 0402WGF1001TCE; footprint Resistor_SMD:R_0603_1608Metric -> Resistor_SMD:R_0402_1005Metric
- R5, R6: value 5.1k -> 0402WGF5101TCE; footprint Resistor_SMD:R_0603_1608Metric -> Resistor_SMD:R_0402_1005Metric
- R7: value 1k -> 0402WGF1001TCE; footprint Resistor_SMD:R_0603_1608Metric -> Resistor_SMD:R_0402_1005Metric
- U3: value NCP1117-3.3_SOT223 -> AMS1117-3.3
Connections:
- net +3V3: now also R4.1; no longer R4.2
- net Col_0: now also U1.30 (GPIO19); no longer U1.7 (GPIO5)
- net Col_1: now also U1.29 (GPIO18); no longer U1.8 (GPIO6)
- net Col_10: now also U1.12 (GPIO9); no longer U1.18 (GPIO15)
- net Col_11: now also U1.11 (GPIO8); no longer U1.27 (GPIO16)
- net Col_12: now also U1.9 (GPIO7); no longer U1.28 (GPIO17)
- net Col_13: now also U1.8 (GPIO6); no longer U1.29 (GPIO18)
- net Col_14: now also U1.7 (GPIO5); no longer U1.30 (GPIO19)
- net Col_2: now also U1.28 (GPIO17); no longer U1.9 (GPIO7)
- net Col_3: now also U1.27 (GPIO16); no longer U1.11 (GPIO8)
- net Col_4: now also U1.18 (GPIO15); no longer U1.12 (GPIO9)
- net Col_5: now also U1.17 (GPIO14); no longer U1.13 (GPIO10)
- net Col_6: now also U1.16 (GPIO13); no longer U1.14 (GPIO11)
- net Col_8: now also U1.14 (GPIO11); no longer U1.16 (GPIO13)
- net Col_9: now also U1.13 (GPIO10); no longer U1.17 (GPIO14)
- net GND: now also SW3.C, SW3.MP, SW3.S2, SW4.C, SW4.MP, SW4.S2
- net RUN: now also R4.2; no longer R4.1
- net SW4_B: now reaches U1.31 (GPIO20)
- net SW4_B: now also SW4.B
- net SW4_A: now reaches U1.32 (GPIO21)
- net SW4_A: now also SW4.A
- net SW4_Button: now reaches U1.34 (GPIO22)
- net SW4_Button: now also SW4.S1
- net SW3_B: now reaches U1.35 (GPIO23)
- net SW3_B: now also SW3.B
- net SW3_A: now reaches U1.36 (GPIO24)
- net SW3_A: now also SW3.A
- net SW3_Button: now reaches U1.37 (GPIO25)
- net SW3_Button: now also SW3.S1
- no-connect marks 14 -> 8
Other:
- moved on the sheet: C14, C15, C16, J1, R5, R6, R7, SW1, SW2, U2, U3

Commit message: stuff
Parts:
- C1, C2: value 0402CG150J500NT -> 0402CG200J500NT
- SW1, SW2: footprint Button_Switch_SMD:SW_Push_1P1T_NO_CK_KMR2 -> Button_Switch_THT:SW_PUSH_1P1T_6x3.5mm_H4.3_APEM_MJTP1243
Connections:
- net GND: now also SW1.2; no longer SW1.1
- net RUN: now also SW1.1; no longer SW1.2
Other:
- moved on the sheet: SW1
Changed lines of the file:
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@@
 	)
 	(junction
+		(at 313.69 185.42)
+		(diameter 0)
+		(color 0 0 0 0)
+	)
+	(junction
 		(at 247.65 125.73)
 		(diameter 0)
@@
 	)
 	(junction
-		(at 213.36 125.73)
+		(at 302.26 129.54)
 		(diameter 0)
 		(color 0 0 0 0)
 	)
 	(junction
-		(at 165.1 146.05)
+		(at 213.36 125.73)
 		(diameter 0)
 		(color 0 0 0 0)
 	)
 	(junction
-		(at 247.65 137.16)
+		(at 165.1 146.05)
 		(diameter 0)
 		(color 0 0 0 0)
 	)
 	(junction
-		(at 213.36 137.16)
+		(at 247.65 137.16)
 		(diameter 0)
 		(color 0 0 0 0)
 	)
 	(junction
-		(at 302.26 129.54)
+		(at 213.36 137.16)
 		(diameter 0)
 		(color 0 0 0 0)
@@
 	)
 	(junction
-		(at 313.69 186.69)
-		(diameter 0)
-		(color 0 0 0 0)
-	)
-	(junction
 		(at 161.29 118.11)
 		(diameter 0)
@@
 	)
 	(junction
-		(at 313.69 191.77)
-		(diameter 0)
-		(color 0 0 0 0)
-	)
-	(junction
 		(at 236.22 125.73)
 		(diameter 0)
@@
 		(color 0 0 0 0)
 	)
+	(junction
+		(at 313.69 190.5)
+		(diameter 0)
+		(color 0 0 0 0)
+	)
 	(no_connect
 		(at 313.69 201.93)
@@
 	(wire
 		(pts
+			(xy 313.69 185.42) (xy 322.58 185.42)
+		)
+		(stroke
+			(width 0)
+			(type default)
+		)
+	)
+	(wire
+		(pts
 			(xy 161.29 116.84) (xy 161.29 118.11)
 		)
@@
 	(wire
 		(pts
+			(xy 313.69 190.5) (xy 322.58 190.5)
+		)
+		(stroke
+			(width 0)
+			(type default)
+		)
+	)
+	(wire
+		(pts
 			(xy 236.22 137.16) (xy 224.79 137.16)
 		)
@@
 	(wire
 		(pts
-			(xy 247.65 137.16) (xy 259.08 137.16)
+			(xy 313.69 190.5) (xy 313.69 191.77)
 		)
 		(stroke
@@
 	(wire
 		(pts
-			(xy 297.18 129.54) (xy 302.26 129.54)
+			(xy 247.65 137.16) (xy 259.08 137.16)
 		)
 		(stroke
@@
 	(wire
 		(pts
-			(xy 313.69 186.69) (xy 322.58 186.69)
-		)
-		(stroke
-			(width 0)
-			(type default)
-		)
-	)
-	(wire
-		(pts
 			(xy 259.08 134.62) (xy 259.08 137.16)
 		)
@@
 	(wire
 		(pts
-			(xy 313.69 184.15) (xy 313.69 186.69)
+			(xy 313.69 184.15) (xy 313.69 185.42)
 		)
 		(stroke
@@
 	(wire
 		(pts
+			(xy 313.69 185.42) (xy 313.69 186.69)
+		)
+		(stroke
+			(width 0)
+			(type default)
+		)
+	)
+	(wire
+		(pts
 			(xy 337.82 133.35) (xy 337.82 143.51)
 		)
@@
 	(wire
 		(pts
-			(xy 313.69 189.23) (xy 313.69 191.77)
+			(xy 313.69 189.23) (xy 313.69 190.5)
 		)
 		(stroke
@@
 	(wire
 		(pts
-			(xy 165.1 134.62) (xy 165.1 146.05)
+			(xy 297.18 129.54) (xy 302.26 129.54)
 		)
 		(stroke
@@
 	(wire
 		(pts
-			(xy 342.9 123.19) (xy 354.33 123.19)
+			(xy 165.1 134.62) (xy 165.1 146.05)
 		)
 		(stroke
@@
 	(wire
 		(pts
-			(xy 181.61 146.05) (xy 182.88 146.05)
+			(xy 342.9 123.19) (xy 354.33 123.19)
 		)
 		(stroke
@@
 	(wire
 		(pts
-			(xy 140.97 118.11) (xy 152.4 118.11)
+			(xy 181.61 146.05) (xy 182.88 146.05)
 		)
 		(stroke
@@
 	(wire
 		(pts
-			(xy 107.95 199.39) (xy 116.84 199.39)
+			(xy 140.97 118.11) (xy 152.4 118.11)
 		)
 		(stroke
@@
 	(wire
 		(pts
-			(xy 247.65 134.62) (xy 247.65 137.16)
+			(xy 107.95 199.39) (xy 116.84 199.39)
 		)
 		(stroke
@@
 	(wire
 		(pts
-			(xy 142.24 171.45) (xy 128.27 171.45)
+			(xy 247.65 134.62) (xy 247.65 137.16)
 		)
 		(stroke
@@
 	(wire
 		(pts
-			(xy 313.69 191.77) (xy 322.58 191.77)
+			(xy 142.24 171.45) (xy 128.27 171.45)
 		)
 		(stroke
@@
 	)
 	(label "USB_D-"
-		(at 322.58 186.69 180)
+		(at 322.58 185.42 180)
 		(fields_autoplaced yes)
 		(effects
@@
 	)
 	(label "USB_D+"
-		(at 322.58 191.77 180)
+		(at 322.58 190.5 180)
 		(fields_autoplaced yes)
 		(effects
@@
 			)
 		)
-		(property "Value" "0402CG150J500NT"
+		(property "Value" "0402CG200J500NT"
 			(at 104.14 193.5511 90)
 			(effects
@@
 			)
 		)
-		(property "Value" "0402CG150J500NT"
+		(property "Value" "0402CG200J500NT"
 			(at 111.76 215.9 90)
 			(effects
@@
 	(symbol
 		(lib_id "Switch:SW_Push")
-		(at 297.18 134.62 90)
+		(at 297.18 134.62 270)
 		(unit 1)
 		(exclude_from_sim no)
@@
 		(fields_autoplaced yes)
 		(property "Reference" "SW1"
-			(at 298.45 133.3499 90)
+			(at 300.99 133.3499 90)
 			(effects
 				(font
 					(size 1.27 1.27)
 				)
-				(justify right)
+				(justify left)
 			)
 		)
 		(property "Value" "SW_Push"
-			(at 298.45 135.8899 90)
+			(at 300.99 135.8899 90)
 			(effects
 				(font
 					(size 1.27 1.27)
 				)
-				(justify right)
+				(justify left)
 			)
 		)
-		(property "Footprint" "Button_Switch_SMD:SW_Push_1P1T_NO_CK_KMR2"
-			(at 292.1 134.62 0)
+		(property "Footprint" "Button_Switch_THT:SW_PUSH_1P1T_6x3.5mm_H4.3_APEM_MJTP1243"
+			(at 302.26 134.62 0)
 			(effects
 				(font
@@
 		)
 		(property "Datasheet" "~"
-			(at 292.1 134.62 0)
+			(at 302.26 134.62 0)
 			(effects
 				(font
@@
 		)
 		(property "Value" "0402WGF5101TCE"
-			(at 328.93 176.276 90)
+			(at 330.2 176.276 90)
 			(effects
 				(font
@@
 		(on_board yes)
 		(dnp no)
-		(fields_autoplaced yes)
 		(property "Reference" "SW2"
 			(at 342.9 135.89 0)
@@
 			)
 		)
-		(property "Footprint" "Button_Switch_SMD:SW_Push_1P1T_NO_CK_KMR2"
+		(property "Footprint" "Button_Switch_THT:SW_PUSH_1P1T_6x3.5mm_H4.3_APEM_MJTP1243"
 			(at 342.9 138.43 0)
 			(effects
