File: pcb/pcb.kicad_pcb (KiCad board)
At the start: 2 copper layers, 293.1 x 126.5 mm, 170 parts, among them J1 USB_C_Receptacle_USB2.0_16P, SW1 SW_SPST, SW10 SW_SPST, SW11 SW_SPST, SW12 SW_SPST, SW13 SW_SPST, SW14 SW_SPST, SW15 SW_SPST, SW16 SW_SPST, SW17 SW_SPST, SW18 SW_SPST, SW19 SW_SPST, SW2 SW_SPST, SW20 SW_SPST, SW21 SW_SPST, SW22 SW_SPST, SW23 SW_SPST, SW24 SW_SPST, SW25 SW_SPST, SW26 SW_SPST, SW27 SW_SPST, SW28 SW_SPST, SW29 SW_SPST, SW3 SW_SPST, SW30 SW_SPST, SW31 SW_SPST, SW32 SW_SPST, SW33 SW_SPST, SW34 SW_SPST, SW35 SW_SPST, SW36 SW_SPST, SW37 SW_SPST, SW38 SW_SPST, SW39 SW_SPST, SW4 SW_SPST, SW40 SW_SPST, SW41 SW_SPST, SW42 SW_SPST, SW43 SW_SPST, SW44 SW_SPST, SW45 SW_SPST, SW46 SW_SPST, SW47 SW_SPST, SW48 SW_SPST, SW49 SW_SPST, SW5 SW_SPST, SW50 SW_SPST, SW51 SW_SPST, SW52 SW_SPST, SW53 SW_SPST, SW54 SW_SPST, SW55 SW_SPST, SW56 SW_SPST, SW57 SW_SPST, SW58 SW_SPST, SW59 SW_SPST, SW6 SW_SPST, SW60 SW_SPST, SW61 SW_SPST, SW62 SW_SPST, SW63 SW_SPST, SW64 SW_SPST, SW65 SW_SPST, SW66 SW_SPST, SW67 SW_SPST, SW68 SW_SPST, SW69 SW_SPST, SW7 SW_SPST, SW8 SW_SPST, SW9 SW_SPST, U1 RP2040, U2 AZ1117-3.3, U3 W25Q128JVS, Y1 YSX321SL

Commit message: add stabilizers
Parts:
- removed H1, H2, H3, H4: MountingHole, MountingHole:MountingHole_3.2mm_M3
- removed SW_BOOTSEL0: SW_Push, Button_Switch_THT:SW_PUSH_6mm_H5mm
- added ST27: Stabilizer, PCM_Mounting_Keyboard_Stabilizer:Stabilizer_Cherry_MX_2.00u, F.Cu at (402.8, 184.3)
- added ST54: Stabilizer, PCM_Mounting_Keyboard_Stabilizer:Stabilizer_Cherry_MX_2.00u, F.Cu at (400.4, 222.4)
- added ST55: Stabilizer, PCM_Mounting_Keyboard_Stabilizer:Stabilizer_Cherry_MX_2.00u, F.Cu at (157.5, 241.4)
- added ST69: Stabilizer, PCM_Mounting_Keyboard_Stabilizer:Stabilizer_Cherry_MX_6.25u, F.Cu at (267.0, 260.5)
- added SWL0: SW_Push, Button_Switch_SMD:SW_Push_1P1T_XKB_TS-1187A, B.Cu at (395.9, 255.0)
- SW27: footprint PCM_Switch_Keyboard_Cherry_MX:SW_Cherry_MX_PCB -> PCM_Switch_Keyboard_Cherry_MX:SW_Cherry_MX_PCB_2.00u
- SW41: footprint PCM_Switch_Keyboard_Cherry_MX:SW_Cherry_MX_PCB -> PCM_Switch_Keyboard_Cherry_MX:SW_Cherry_MX_PCB_1.50u
- SW55: footprint PCM_Switch_Keyboard_Cherry_MX:SW_Cherry_MX_PCB -> PCM_Switch_Keyboard_Cherry_MX:SW_Cherry_MX_PCB_2.25u
Routing:
- net /ROW1: track 371.5 -> 376.0 mm
- net /COL3: track 328.3 -> 324.6 mm
- net /COL2: track 330.3 -> 326.7 mm
- net /COL1: track 368.2 -> 364.8 mm
- net GND: track 43.2 -> 46.4 mm, vias 30 -> 29
- net /ROW2: track 343.7 -> 341.8 mm
- net /QSPI_SS: track 17.1 -> 16.5 mm
Other:
- board text removed: "25.4"
