File: pcb/pcb.kicad_sch (KiCad schematic)
At the start: 170 parts, among them J1 USB_C_Receptacle_USB2.0_16P, SW1 SW_SPST, SW10 SW_SPST, SW11 SW_SPST, SW12 SW_SPST, SW13 SW_SPST, SW14 SW_SPST, SW15 SW_SPST, SW16 SW_SPST, SW17 SW_SPST, SW18 SW_SPST, SW19 SW_SPST, SW2 SW_SPST, SW20 SW_SPST, SW21 SW_SPST, SW22 SW_SPST, SW23 SW_SPST, SW24 SW_SPST, SW25 SW_SPST, SW26 SW_SPST, SW27 SW_SPST, SW28 SW_SPST, SW29 SW_SPST, SW3 SW_SPST, SW30 SW_SPST, SW31 SW_SPST, SW32 SW_SPST, SW33 SW_SPST, SW34 SW_SPST, SW35 SW_SPST, SW36 SW_SPST, SW37 SW_SPST, SW38 SW_SPST, SW39 SW_SPST, SW4 SW_SPST, SW40 SW_SPST, SW41 SW_SPST, SW42 SW_SPST, SW43 SW_SPST, SW44 SW_SPST, SW45 SW_SPST, SW46 SW_SPST, SW47 SW_SPST, SW48 SW_SPST, SW49 SW_SPST, SW5 SW_SPST, SW50 SW_SPST, SW51 SW_SPST, SW52 SW_SPST, SW53 SW_SPST, SW54 SW_SPST, SW55 SW_SPST, SW56 SW_SPST, SW57 SW_SPST, SW58 SW_SPST, SW59 SW_SPST, SW6 SW_SPST, SW60 SW_SPST, SW61 SW_SPST, SW62 SW_SPST, SW63 SW_SPST, SW64 SW_SPST, SW65 SW_SPST, SW66 SW_SPST, SW67 SW_SPST, SW68 SW_SPST, SW69 SW_SPST, SW7 SW_SPST, SW8 SW_SPST, SW9 SW_SPST, U1 RP2040, U2 AZ1117-3.3, U3 W25Q128JVS, Y1 YSX321SL

Commit message: add stabilizers
Parts:
- removed H1, H2, H3, H4: MountingHole, MountingHole:MountingHole_3.2mm_M3, symbol Mechanical:MountingHole
- added ST27, ST54, ST55: Stabilizer, PCM_Mounting_Keyboard_Stabilizer:Stabilizer_Cherry_MX_2.00u, symbol Mechanical:MountingHole
- added ST69: Stabilizer, PCM_Mounting_Keyboard_Stabilizer:Stabilizer_Cherry_MX_6.25u, symbol Mechanical:MountingHole
- C10, C11: LCSC (none) -> C52923
- C12, C13, C14, C3, C4, C5, C6, C7, C8, C9: LCSC (none) -> C1525
- C15, C16: LCSC (none) -> C1658
- C2: LCSC (none) -> C19702
- D1, D10, D11, D12, D13, D14, D15, D16, D17, D18, D19, D2, D20, D21, D22, D23, D24, D25, D26, D27, D28, D29, D3, D30, D31, D32, D33, D34, D35, D36, D37, D38, D39, D4, D40, D41, D42, D43, D44, D45, D46, D47, D48, D49, D5, D50, D51, D52, D53, D54, D55, D56, D57, D58, D59, D6, D60, D61, D62, D63, D64, D65, D66, D67, D68, D69, D7, D8, D9: LCSC (none) -> C2128
- J1: LCSC (none) -> C2927037
- R1, R2: LCSC (none) -> C25905
- R3: LCSC (none) -> C25744
- R5, R6: LCSC (none) -> C25092
- SW27: footprint PCM_Switch_Keyboard_Cherry_MX:SW_Cherry_MX_PCB -> PCM_Switch_Keyboard_Cherry_MX:SW_Cherry_MX_PCB_2.00u
- SW41: footprint PCM_Switch_Keyboard_Cherry_MX:SW_Cherry_MX_PCB -> PCM_Switch_Keyboard_Cherry_MX:SW_Cherry_MX_PCB_1.50u
- SW55: footprint PCM_Switch_Keyboard_Cherry_MX:SW_Cherry_MX_PCB -> PCM_Switch_Keyboard_Cherry_MX:SW_Cherry_MX_PCB_2.25u
- SWL0: renamed from SW_BOOTSEL0; footprint Button_Switch_THT:SW_PUSH_6mm_H5mm -> Button_Switch_SMD:SW_Push_1P1T_XKB_TS-1187A; LCSC (none) -> C318884
- U1: LCSC (none) -> C2040
- U2: LCSC (none) -> C6186
- U3: LCSC (none) -> C97521
